File: Catch The Light Game.brd (EAGLE design)
At the start: 90.2 x 98.7 mm, 43 parts, among them J2 J3MM, J3 J15MM, J5 J20MM, J6 J7MM, J7 J5MM, Q1 16 MHz, U1 ATMEGA328PB-AU, X1 MINI-USB-SCHIELD-32005-201

Commit message: Add files via upload
Parts:
- added C1: 100 nf, rcl:C025-024X044
- added C4: 10 nf, rcl:C025-024X044
- moved GND 11.4 mm to (82.5, 67.3)
- moved J5 2.54 mm to (67.3, 54.6)
- moved J6 2.54 mm to (77.5, 73.7)
- moved JP1 1.27 mm to (83.8, 49.5)
Connections:
- net 0: now also C1.1, C4.1
- net VCC: now also C1.2, C4.2
Routing:
- net N$53: track 2.54 -> 17.8 mm
- net 0: track 282.0 -> 295.6 mm
- net VCC: track 122.8 -> 134.3 mm
- net N$27: track 48.1 -> 36.7 mm
- net N$56: track 36.8 -> 39.4 mm
- net N$48: track 2.54 -> 5.08 mm
- net N$8: track 18.4 -> 19.7 mm
- net N$54: track 3.81 -> 5.08 mm
- net N$32: track 18.4 -> 19.7 mm
- net N$46: track 26.7 -> 27.9 mm
Other:
- board text added: "10 nf"
- board text added: "100 nf"
